File: pcbs/frame_corners/frame_corners.kicad_pcb (KiCad board)
At the start: 2 copper layers, 55 x 40 mm, 8 parts

Commit message: Panelization with https://gitlab.com/dren.dk/kicad-util
Parts:
- removed the REF** at (-398.6, -540.0)
- removed the REF** at (-390.0, -548.6)
- added REF**: PinHeader_2x05_P2.54mm_Vertical, Connector_PinHeader_2.54mm:PinHeader_2x05_P2.54mm_Vertical, F.Cu at (145.3, 99.0)
- added REF**: PinHeader_2x05_P2.54mm_Vertical, Connector_PinHeader_2.54mm:PinHeader_2x05_P2.54mm_Vertical, B.Cu at (153.5, 90.8)
- moved REF** 839.2 mm to (170.3, 90.8)
- moved REF** 839.2 mm to (145.3, 115.8)
- moved REF** 838.9 mm to (167.5, 95.0)
- moved REF** 838.9 mm to (149.5, 95.0)
- moved REF** 838.9 mm to (191.3, 95.0)
- moved REF** 838.9 mm to (149.5, 113.0)
Other:
- board size 55 x 40 mm -> 53.6 x 40 mm
